File: circuit/circuit.sch (KiCad schematic (older format))
At the start: 8 parts

Commit message: Pushing the changes to the schematic
Parts:
- removed U?: ADXL345, footprints:ADXL345, symbol formula:ADXL345
- added C1, C2: C_30pF, footprints:C_0805_OEM, symbol formula:C_30pF
- added U1: MIC5504-3.3YM5, Package_TO_SOT_SMD:SOT-23-5, symbol Regulator_Linear:MIC5504-3.3YM5
- added U2: ADXL345, footprints:ADXL345, symbol formula:ADXL345
- added Y1: Crystal_SMD, footprints:Crystal_SMD_FA238, symbol formula:Crystal_SMD
- gave numbers to parts that had none: 7
Connections:
- net labels added: Digital_Interface_Supply_Voltage, Enable_Input, P_LED_1, P_LED_2, P_LED_3, RESET, Slave_Select, chip_select, miso, mosi, sck
- wire segments 8 -> 77
- no-connect marks 0 -> 14
Other:
- moved on the sheet: U3

Commit message: updated schematic
Parts:
- added J?: UF_2_RA, footprints:Ultrafit_2_RA, symbol formula:UF_2_RA
- added J?: CONN_02X03, footprints:Pin_Header_Straight_2x03, symbol formula:CONN_02X03
- added R? (x3): R_200, footprints:R_0805_OEM, symbol formula:R_200
Connections:
- net labels added: Battery+, INT1, INT2
- net labels removed: Digital_Interface_Supply_Voltage, Enable_Input, chip_select
- wire segments 77 -> 73

Commit message: Version one of the schematic with footprints
Parts:
- gave numbers to parts that had none: 5
Changed lines of the file:
@@
 Battery+
 $Comp
-L formula:R_200 R?
+L formula:R_200 R4
 U 1 1 5C5A80DD
 P 2650 3900
-F 0 "R?" H 2700 4100 50  0000 L CNN
+F 0 "R4" H 2700 4100 50  0000 L CNN
 F 1 "R_200" H 2300 3850 50  0000 L CNN
 F 2 "footprints:R_0805_OEM" H 2580 3900 50  0001 C CNN
@@
 $EndComp
 $Comp
-L formula:R_200 R?
+L formula:R_200 R3
 U 1 1 5C5A821D
 P 2450 3900
-F 0 "R?" H 2500 4100 50  0000 L CNN
+F 0 "R3" H 2500 4100 50  0000 L CNN
 F 1 "R_200" H 2750 3850 50  0000 L CNN
 F 2 "footprints:R_0805_OEM" H 2380 3900 50  0001 C CNN
@@
 $EndComp
 $Comp
-L formula:R_200 R?
+L formula:R_200 R2
 U 1 1 5C5A8292
 P 2250 3900
-F 0 "R?" H 2300 4100 50  0000 L CNN
+F 0 "R2" H 2300 4100 50  0000 L CNN
 F 1 "R_200" H 2350 3950 50  0000 L CNN
 F 2 "footprints:R_0805_OEM" H 2180 3900 50  0001 C CNN
@@
 $EndComp
 $Comp
-L power:GND #PWR?
+L power:GND #PWR013
 U 1 1 5C5A859C
 P 2650 4050
-F 0 "#PWR?" H 2650 3800 50  0001 C CNN
+F 0 "#PWR013" H 2650 3800 50  0001 C CNN
 F 1 "GND" H 2655 3877 50  0000 C CNN
 F 2 "" H 2650 4050 50  0001 C CNN
@@
 $EndComp
 $Comp
-L power:GND #PWR?
+L power:GND #PWR012
 U 1 1 5C5AC273
 P 2450 4050
-F 0 "#PWR?" H 2450 3800 50  0001 C CNN
+F 0 "#PWR012" H 2450 3800 50  0001 C CNN
 F 1 "GND" H 2455 3877 50  0000 C CNN
 F 2 "" H 2450 4050 50  0001 C CNN
@@
 $EndComp
 $Comp
-L power:GND #PWR?
+L power:GND #PWR02
 U 1 1 5C5AE078
 P 2250 4050
-F 0 "#PWR?" H 2250 3800 50  0001 C CNN
+F 0 "#PWR02" H 2250 3800 50  0001 C CNN
 F 1 "GND" H 2255 3877 50  0000 C CNN
 F 2 "" H 2250 4050 50  0001 C CNN
@@
 	4400 4000 4400 4100
 $Comp
-L power:VCC #PWR?
+L power:VCC #PWR015
 U 1 1 5C5B59C6
 P 4000 3450
-F 0 "#PWR?" H 4000 3300 50  0001 C CNN
+F 0 "#PWR015" H 4000 3300 50  0001 C CNN
 F 1 "VCC" H 4017 3623 50  0000 C CNN
 F 2 "" H 4000 3450 50  0001 C CNN
@@
 	3900 1300 4500 1300
 $Comp
-L power:VCC #PWR?
+L power:VCC #PWR014
 U 1 1 5C5B9935
 P 3900 1150
-F 0 "#PWR?" H 3900 1000 50  0001 C CNN
+F 0 "#PWR014" H 3900 1000 50  0001 C CNN
 F 1 "VCC" H 3917 1323 50  0000 C CNN
 F 2 "" H 3900 1150 50  0001 C CNN
@@
 	5400 1100 5400 1300
 $Comp
-L formula:UF_2_RA J?
+L formula:UF_2_RA J1
 U 1 1 5C5BC0BF
 P 1550 1400
-F 0 "J?" H 1606 1697 60  0000 C CNN
+F 0 "J1" H 1606 1697 60  0000 C CNN
 F 1 "UF_2_RA" H 1606 1591 60  0000 C CNN
 F 2 "footprints:Ultrafit_2_RA" H 1450 1450 60  0001 C CNN
@@
 	1900 1450 1900 1550
 $Comp
-L power:GND #PWR?
+L power:GND #PWR01
 U 1 1 5C5CFFAC
 P 1900 1550
-F 0 "#PWR?" H 1900 1300 50  0001 C CNN
+F 0 "#PWR01" H 1900 1300 50  0001 C CNN
 F 1 "GND" H 1905 1377 50  0000 C CNN
 F 2 "" H 1900 1550 50  0001 C CNN
@@
 $EndComp
 $Comp
-L formula:CONN_02X03 J?
+L formula:CONN_02X03 J2
 U 1 1 5C5D0C55
 P 4900 2350
-F 0 "J?" H 4900 2665 50  0000 C CNN
+F 0 "J2" H 4900 2665 50  0000 C CNN
 F 1 "CONN_02X03" H 4900 2574 50  0000 C CNN
 F 2 "footprints:Pin_Header_Straight_2x03" H 4900 1150 50  0001 C CNN
@@
 	5400 2250 5400 2150
 $Comp
-L power:VCC #PWR?
+L power:VCC #PWR017
 U 1 1 5C5D2E9C
 P 5400 2150
-F 0 "#PWR?" H 5400 2000 50  0001 C CNN
+F 0 "#PWR017" H 5400 2000 50  0001 C CNN
 F 1 "VCC" H 5417 2323 50  0000 C CNN
 F 2 "" H 5400 2150 50  0001 C CNN
@@
 	5250 2450 5250 2600
 $Comp
-L power:GND #PWR?
+L power:GND #PWR016
 U 1 1 5C5D503B
 P 5250 2600
-F 0 "#PWR?" H 5250 2350 50  0001 C CNN
+F 0 "#PWR016" H 5250 2350 50  0001 C CNN
 F 1 "GND" H 5255 2427 50  0000 C CNN
 F 2 "" H 5250 2600 50  0001 C CNN

Commit message: schematic edited
Parts:
- added C? (x2): C_30pF, footprints:C_0805_OEM, symbol formula:C_30pF
- added J?: Micro_SD_Card, symbol Connector:Micro_SD_Card
- added R?: R_200, footprints:R_0805_OEM, symbol formula:R_200
- added U?: SK812, footprints:SK6812, symbol formula:SK812
Connections:
- net labels added: Neopix, SD_Select
- wire segments 73 -> 81
- no-connect marks 14 -> 12
Other:
- moved on the sheet: U3

Commit message: We can final make the layout
Parts:
- removed J1: UF_2_RA, footprints:Ultrafit_2_RA, symbol formula:UF_2_RA
- removed J?: Micro_SD_Card, symbol Connector:Micro_SD_Card
- removed R4: R_200, footprints:R_0805_OEM, symbol formula:R_200
- added C7: C_1uF, footprints:C_0805_OEM, symbol formula:C_1uF
- added J1: JST-PH_2_RA, footprints:JST-PH_2_RA, symbol formula:JST-PH_2_RA
- added R5, R7: R_10K, footprints:R_0805_OEM, symbol formula:R_10K
- added R6: R_200, footprints:R_0805_OEM, symbol formula:R_200
- added SD1: Micro_SD_Card_A118117CT-ND, footprints:Micro_SD_Card_A118117CT-ND, symbol formula:Micro_SD_Card_A118117CT-ND
- added U5: ATmega328P-AU, Package_QFP:TQFP-32_7x7mm_P0.8mm, symbol MCU_Microchip_ATmega:ATmega328P-AU
- gave numbers to parts that had none: 4
Connections:
- net labels added: cardIN
- net labels removed: P_LED_2, P_LED_3
- wire segments 81 -> 85
- no-connect marks 12 -> 20

Commit message: oh geez. windows and ubuntu
Parts:
- removed J1: JST-PH_2_RA, footprints:JST-PH_2_RA, symbol formula:JST-PH_2_RA
- removed J2: CONN_02X03, footprints:Pin_Header_Straight_2x03, symbol formula:CONN_02X03
- removed SD1: Micro_SD_Card_A118117CT-ND, footprints:Micro_SD_Card_A118117CT-ND, symbol formula:Micro_SD_Card_A118117CT-ND
- removed U2: ADXL345, footprints:ADXL345, symbol formula:ADXL345
- removed U3, U5: ATmega328P-AU, Package_QFP:TQFP-32_7x7mm_P0.8mm, symbol MCU_Microchip_ATmega:ATmega328P-AU
- removed U4: SK812, footprints:SK6812, symbol formula:SK812
- added J1: JST-PH_2_RA, rocketry:JST-PH_2_RA, symbol rocketry:JST-PH_2_RA
- added J2: CONN_02X03, rocketry:Pin_Header_Straight_2x03, symbol rocketry:CONN_02X03
- added SD1: Micro_SD_Card_A118117CT-ND, rocketry:Micro_SD_Card_A118117CT-ND, symbol rocketry:Micro_SD_Card_A118117CT-ND
- added U1: SK812, rocketry:SK6812, symbol rocketry:SK812
- added U3: ADXL345, rocketry:ADXL345, symbol rocketry:ADXL345
- added U4: ATmega328-AU, rocketry:TQFP-32_7x7mm_Pitch0.8mm, symbol MCU_Microchip_ATmega:ATmega328-AU
- C1: renamed from C7; footprint footprints:C_0805_OEM -> rocketry:C_0805_OEM
- C2: renamed from C5; footprint footprints:C_0805_OEM -> rocketry:C_0805_OEM
- C3: renamed from C6; footprint footprints:C_0805_OEM -> rocketry:C_0805_OEM
- C4: renamed from C1; footprint footprints:C_0805_OEM -> rocketry:C_0805_OEM
- C5: renamed from C2; footprint footprints:C_0805_OEM -> rocketry:C_0805_OEM
- C6: renamed from C3; footprint footprints:C_0805_OEM -> rocketry:C_0805_OEM
- C7: renamed from C4; footprint footprints:C_0805_OEM -> rocketry:C_0805_OEM
- D1: footprint footprints:LED_0805_OEM -> rocketry:LED_0805_OEM
- D2: renamed from D3; footprint footprints:LED_0805_OEM -> rocketry:LED_0805_OEM
- D3: renamed from D2; footprint footprints:LED_0805_OEM -> rocketry:LED_0805_OEM
- R1: renamed from R2; footprint footprints:R_0805_OEM -> rocketry:R_0805_OEM
- R2: renamed from R6; footprint footprints:R_0805_OEM -> rocketry:R_0805_OEM
- R3: footprint footprints:R_0805_OEM -> rocketry:R_0805_OEM
- R4: renamed from R5; footprint footprints:R_0805_OEM -> rocketry:R_0805_OEM
- R5: renamed from R4; footprint footprints:R_0805_OEM -> rocketry:R_0805_OEM
- R6: renamed from R7; footprint footprints:R_0805_OEM -> rocketry:R_0805_OEM
- R7: renamed from R1; footprint footprints:R_0805_OEM -> rocketry:R_0805_OEM
- U2: renamed from U1; footprint Package_TO_SOT_SMD:SOT-23-5 -> rocketry:SOT-23-5_OEM
- Y1: footprint footprints:Crystal_SMD_FA238 -> rocketry:Crystal_SMD_FA238
Connections:
- wire segments 85 -> 74
- no-connect marks 20 -> 17

Commit message: modified schematic and layout:
Parts:
- removed C2, C3: C_30pF, rocketry:C_0805_OEM, symbol formula:C_30pF
- removed J2: CONN_02X03, rocketry:Pin_Header_Straight_2x03, symbol rocketry:CONN_02X03
- removed U2: MIC5504-3.3YM5, rocketry:SOT-23-5_OEM, symbol Regulator_Linear:MIC5504-3.3YM5
- added C2: C_10uF, footprints:C_0805_OEM, symbol rocketry:C_10uF
- added C3: C_100uF, footprints:C_0805_OEM, symbol rocketry:C_100uF
- added C8: C_1uF, footprints:C_0805_OEM, symbol rocketry:C_1uF
- added C9: C_0.1uF, footprints:C_0805_OEM, symbol rocketry:C_0.1uF
- added U2: LM1117-3.3, TO_SOT_Packages_SMD:SOT-223, symbol rocketry:LM1117-3.3
- added U5: USB_MicroB, Connectors_USB:USB_Micro-B_Molex-105017-0001, symbol rocketry:USB_MicroB
Connections:
- wire segments 74 -> 76

Commit message: revision two
Parts:
- removed C2: C_10uF, footprints:C_0805_OEM, symbol rocketry:C_10uF
- removed C3: C_100uF, footprints:C_0805_OEM, symbol rocketry:C_100uF
- removed U2: LM1117-3.3, TO_SOT_Packages_SMD:SOT-223, symbol rocketry:LM1117-3.3
- added C2: C_0.1uF, footprints:C_0805_OEM, symbol formula:C_0.1uF
- added C3: C_1uF, footprints:C_0805_OEM, symbol formula:C_1uF
- added R10, R8: R_4.7K, footprints:R_0805_OEM, symbol rocketry:R_4.7K
- added R11, R9: R_10K, footprints:R_0805_OEM, symbol rocketry:R_10K
- added U2: TCR2EF33LM, rocketry:SOT25, symbol rocketry:TCR2EF33LM
- added U6: 4050_Logic_Buffer, Housings_SOIC:SOIC-16_3.9x9.9mm_Pitch1.27mm, symbol rocketry:4050_Logic_Buffer
Connections:
- net labels added: MISO, MISO_3V, MOSI, MOSI_3V, SCK, SCK_3V, SCL, SCL_3V, SDA, SDA_3V, SD_CS, SD_CS_3V
- net labels removed: SD_Select, Slave_Select, miso, mosi, sck
- wire segments 76 -> 86
- no-connect marks 17 -> 18
