File: circuit/circuit.sch (KiCad schematic (older format))
At the start: 32 parts, among them J1 JST-PH_2_RA, U1 SK812, U2 TCR2EF33LM, U3 ADXL345, U4 ATmega328-AU, U5 USB_MicroB, U6 4050_Logic_Buffer, Y1 Crystal_SMD

Commit message: starting rev 3
Parts:
- removed C2: C_0.1uF, footprints:C_0805_OEM, symbol formula:C_0.1uF
- removed C3: C_1uF, footprints:C_0805_OEM, symbol formula:C_1uF
- removed R10, R8: R_4.7K, footprints:R_0805_OEM, symbol rocketry:R_4.7K
- removed U2: TCR2EF33LM, rocketry:SOT25, symbol rocketry:TCR2EF33LM
- removed U6: 4050_Logic_Buffer, Housings_SOIC:SOIC-16_3.9x9.9mm_Pitch1.27mm, symbol rocketry:4050_Logic_Buffer
- added C2, C3: C_10uF, footprints:C_0805_OEM, symbol rocketry:C_10uF
- added R? (x2): R_10K, footprints:R_0805_OEM, symbol rocketry:R_10K
- added U2: LM1117MPX-3.3, TO_SOT_Packages_SMD:SOT-223, symbol rocketry:LM1117MPX-3.3
Connections:
- net labels removed: SCL_3V, SDA_3V
- wire segments 86 -> 84
- no-connect marks 18 -> 16

Commit message: working on rev3
Parts:
- removed R4: R_10K, rocketry:R_0805_OEM, symbol formula:R_10K
- removed SD1: Micro_SD_Card_A118117CT-ND, rocketry:Micro_SD_Card_A118117CT-ND, symbol rocketry:Micro_SD_Card_A118117CT-ND
- added SD1: MicroSD_V2, rocketry:Micro_SD_Card_Holder_Molex, symbol rocketry:MicroSD_V2
- gave numbers to parts that had none: 2
Connections:
- net labels added: Dectect_LED
- net labels removed: MISO_3V, MOSI_3V, SCK_3V, SD_CS_3V, cardIN
- wire segments 84 -> 80
Changed lines of the file:
@@
-	-1   0    0    -1
-$EndComp
-Text Label 8675 5500 2    50   ~ 0
-SCK_3V
-Text Label 8675 5700 2    50   ~ 0
-MISO_3V
-$Comp
-L power:VCC #PWR0121
-U 1 1 5C64965B
-P 8250 5250
-F 0 "#PWR0121" H 8250 5100 50  0001 C CNN
-F 1 "VCC" H 8267 5423 50  0000 C CNN
-F 2 "" H 8250 5250 50  0001 C CNN
-F 3 "" H 8250 5250 50  0001 C CNN
-	1    8250 5250
-	-1   0    0    -1
-$EndComp
-$Comp
-L power:GND #PWR0122
-U 1 1 5C649692
-P 8125 5900
-F 0 "#PWR0122" H 8125 5650 50  0001 C CNN
-F 1 "GND" H 8130 5727 50  0000 C CNN
-F 2 "" H 8125 5900 50  0001 C CNN
-F 3 "" H 8125 5900 50  0001 C CNN
-	1    8125 5900
 	-1   0    0    -1
 $EndComp
@@
 	-1   0    0    -1
 $EndComp
-$Comp
-L formula:R_10K R4
-U 1 1 5C65F207
-P 1700 7200
-F 0 "R4" H 1770 7246 50  0000 L CNN
-F 1 "R_10K" H 1770 7155 50  0000 L CNN
-F 2 "rocketry:R_0805_OEM" H 1630 7200 50  0001 C CNN
-F 3 "http://www.bourns.com/data/global/pdfs/CRS.pdf" H 1780 7200 50  0001 C CNN
-F 4 "DK" H 1700 7200 60  0001 C CNN "MFN"
-F 5 "CRS0805-FX-1002ELFCT-ND" H 1700 7200 60  0001 C CNN "MPN"
-F 6 "https://www.digikey.com/products/en?keywords=CRS0805-FX-1002ELFCT-ND" H 2180 7600 60  0001 C CNN "PurchasingLink"
-	1    1700 7200
-	-1   0    0    -1
-$EndComp
-$Comp
-L power:GND #PWR0124
-U 1 1 5C66A2FF
-P 1700 7350
-F 0 "#PWR0124" H 1700 7100 50  0001 C CNN
-F 1 "GND" H 1705 7177 50  0000 C CNN
-F 2 "" H 1700 7350 50  0001 C CNN
-F 3 "" H 1700 7350 50  0001 C CNN
-	1    1700 7350
-	-1   0    0    -1
-$EndComp
 Wire Wire Line
 	1000 6900 1000 7250
-Wire Wire Line
-	1700 7050 1700 6900
-Wire Wire Line
-	1750 6900 1700 6900
-Connection ~ 1700 6900
-Wire Wire Line
-	1700 6900 1600 6900
-$Comp
-L power:VCC #PWR0125
-U 1 1 5C6735B4
-P 8350 5775
-F 0 "#PWR0125" H 8350 5625 50  0001 C CNN
-F 1 "VCC" H 8450 5800 50  0000 C CNN
-F 2 "" H 8350 5775 50  0001 C CNN
-F 3 "" H 8350 5775 50  0001 C CNN
-	1    8350 5775
-	-1   0    0    -1
-$EndComp
-Text Label 8675 6000 2    50   ~ 0
-cardIN
-Text Label 1750 6900 0    50   ~ 0
-cardIN
-Text Label 9825 1525 2    50   ~ 0
-cardIN
 $Comp
 L formula:R_10K R6
@@
 	9475 3025 9825 3025
 NoConn ~ 9825 3625
-NoConn ~ 8675 5100
-NoConn ~ 8675 5800
 NoConn ~ 11025 1525
 NoConn ~ 11025 1725
 NoConn ~ 11025 1825
-Wire Wire Line
-	8675 5400 8250 5400
-Wire Wire Line
-	8250 5400 8250 5250
-Wire Wire Line
-	8350 5775 8350 5900
-Wire Wire Line
-	8350 5900 8675 5900
-Wire Wire Line
-	8675 5600 8125 5600
-Wire Wire Line
-	8125 5600 8125 5900
-$Comp
-L rocketry:Micro_SD_Card_A118117CT-ND SD1
-U 1 1 5C6B510A
-P 9575 5550
-F 0 "SD1" H 10404 5687 50  0000 L CNN
-F 1 "Micro_SD_Card_A118117CT-ND" H 10404 5596 50  0000 L CNN
-F 2 "rocketry:Micro_SD_Card_A118117CT-ND" H 9625 6800 50  0001 C CNN
-F 3 "https://www.te.com/commerce/DocumentDelivery/DDEController?Action=srchrtrv&DocNm=2201778&DocType=Customer+Drawing&DocLang=JP" H 9675 6450 50  0001 C CNN
-F 4 "A118117CT-ND" H 10404 5505 50  0000 L CNN "Digi-Key Part Number"
-F 5 "2201778-1" H 10404 5414 50  0000 L CNN "MPN"
-	1    9575 5550
-	1    0    0    -1
-$EndComp
 $Comp
 L rocketry:SK812 U1
@@
 	1    0    0    -1
 $EndComp
-Wire Wire Line
-	1375 2450 1475 2450
 Wire Wire Line
 	4075 2750 4075 2850
@@
 	4050 5925 4050 5750
 Connection ~ 3500 5925
-Text Label 8675 5300 2    50   ~ 0
-MOSI_3V
-Wire Wire Line
-	10425 675  10325 675
 Wire Wire Line
 	10425 675  10425 1025
-Text Label 10325 675  2    50   ~ 0
-Battery+
-Text Label 1475 2450 0    50   ~ 0
-Battery+
 Wire Wire Line
 	5525 2700 5525 2550
@@
 	1    0    0    -1
 $EndComp
-Text Label 8675 5200 2    50   ~ 0
-SD_CS_3V
 Text Label 9825 1925 2    50   ~ 0
 MISO
@@
 SCL
 NoConn ~ 9825 2425
-Text Label 4050 5750 0    50   ~ 0
-Battery+
-Text Label 9125 2825 2    50   ~ 0
-Battery+
 $Comp
 L rocketry:LM1117MPX-3.3 U2
@@
 	3225 1500 3225 1675
 $Comp
-L rocketry:R_10K R?
+L rocketry:R_10K R4
 U 1 1 5CB428D3
 P 5525 2400
-F 0 "R?" H 5595 2446 50  0000 L CNN
+F 0 "R4" H 5595 2446 50  0000 L CNN
 F 1 "R_10K" H 5595 2355 50  0000 L CNN
 F 2 "footprints:R_0805_OEM" H 5455 2400 50  0001 C CNN
@@
 $EndComp
 $Comp
-L rocketry:R_10K R?
+L rocketry:R_10K R8
 U 1 1 5CB429A6
 P 5975 2400
-F 0 "R?" H 6045 2446 50  0000 L CNN
+F 0 "R8" H 6045 2446 50  0000 L CNN
 F 1 "R_10K" H 6045 2355 50  0000 L CNN
 F 2 "footprints:R_0805_OEM" H 5905 2400 50  0001 C CNN
@@
 	1    0    0    -1
 $EndComp
+NoConn ~ 7900 5125
+Text Label 7900 5325 2    50   ~ 0
+MOSI
+$Comp
+L power:VCC #PWR013
+U 1 1 5CB6F2B9
+P 7275 5200
+F 0 "#PWR013" H 7275 5050 50  0001 C CNN
+F 1 "VCC" H 7292 5373 50  0000 C CNN
+F 2 "" H 7275 5200 50  0001 C CNN
+F 3 "" H 7275 5200 50  0001 C CNN
+	1    7275 5200
+	-1   0    0    -1
+$EndComp
+Text Label 7900 5225 2    50   ~ 0
+SD_CS
+Wire Wire Line
+	7900 5425 7275 5425
+Wire Wire Line
+	7275 5425 7275 5200
+Text Label 7900 5525 2    50   ~ 0
+SCK
+$Comp
+L power:GND #PWR012
+U 1 1 5CB7648D
+P 7000 5725
+F 0 "#PWR012" H 7000 5475 50  0001 C CNN
+F 1 "GND" H 7005 5552 50  0000 C CNN
+F 2 "" H 7000 5725 50  0001 C CNN
+F 3 "" H 7000 5725 50  0001 C CNN
+	1    7000 5725
+	-1   0    0    -1
+$EndComp
+Wire Wire Line
+	7900 5625 7000 5625
+Wire Wire Line
+	7000 5625 7000 5725
+Text Label 7900 5725 2    50   ~ 0
+MISO
+$Comp
+L rocketry:MicroSD_V2 SD1
+U 1 1 5CB6A124
+P 8800 5575
+F 0 "SD1" H 9629 5621 50  0000 L CNN
+F 1 "MicroSD_V2" H 9629 5530 50  0000 L CNN
+F 2 "rocketry:Micro_SD_Card_Holder_Molex" H 8850 6825 50  0001 C CNN
+F 3 "https://www.te.com/commerce/DocumentDelivery/DDEController?Action=srchrtrv&DocNm=2201778&DocType=Customer+Drawing&DocLang=JP" H 8900 6475 50  0001 C CNN
+F 4 "https://www.digikey.com/product-detail/en/molex/0473521001/WM3290CT-ND/2405698" H 9100 6675 50  0001 C CNN "Purchasing Link"
+F 5 "WM3290CT-ND" H 8800 6575 50  0001 C CNN "Digi-Key Part Number"
+F 6 "0473521001" H 8800 6675 50  0001 C CNN "MPN"
+	1    8800 5575
+	1    0    0    -1
+$EndComp
+NoConn ~ 7900 5825
+Wire Wire Line
+	1600 6900 1750 6900
+Text Label 1750 6900 0    50   ~ 0
+Dectect_LED
+Text Label 7900 5925 2    50   ~ 0
+Dectect_LED
+$Comp
+L power:VCC #PWR011
+U 1 1 5CB8BA57
+P 4050 5750
+F 0 "#PWR011" H 4050 5600 50  0001 C CNN
+F 1 "VCC" H 4067 5923 50  0000 C CNN
+F 2 "" H 4050 5750 50  0001 C CNN
+F 3 "" H 4050 5750 50  0001 C CNN
+	1    4050 5750
+	-1   0    0    -1
+$EndComp
+$Comp
+L power:VCC #PWR015
+U 1 1 5CB8BC42
+P 10425 675
+F 0 "#PWR015" H 10425 525 50  0001 C CNN
+F 1 "VCC" H 10442 848 50  0000 C CNN
+F 2 "" H 10425 675 50  0001 C CNN
+F 3 "" H 10425 675 50  0001 C CNN
+	1    10425 675
+	1    0    0    -1
+$EndComp
+$Comp
+L power:VCC #PWR014
+U 1 1 5CB8BFB3
+P 9125 2825
+F 0 "#PWR014" H 9125 2675 50  0001 C CNN
+F 1 "VCC" H 9142 2998 50  0000 C CNN
+F 2 "" H 9125 2825 50  0001 C CNN
+F 3 "" H 9125 2825 50  0001 C CNN
+	1    9125 2825
+	1    0    0    -1
+$EndComp
+$Comp
+L power:VCC #PWR06
+U 1 1 5CB8C32E
+P 1625 2375
+F 0 "#PWR06" H 1625 2225 50  0001 C CNN
+F 1 "VCC" H 1642 2548 50  0000 C CNN
+F 2 "" H 1625 2375 50  0001 C CNN
+F 3 "" H 1625 2375 50  0001 C CNN
+	1    1625 2375
+	1    0    0    -1
+$EndComp
+Wire Wire Line
+	1625 2450 1625 2375
+Wire Wire Line
+	1375 2450 1625 2450
+Text Label 9825 1525 2    50   ~ 0
+Dectect_LED
+Text Label 5975 2800 0    50   ~ 0
+SDA
+Text Label 5525 2700 0    50   ~ 0
+SCL
 $EndSCHEMATC

Commit message: Schematic with a 2x03 connector
Parts:
- removed U5: USB_MicroB, Connectors_USB:USB_Micro-B_Molex-105017-0001, symbol rocketry:USB_MicroB
- added J2: CONN_02X03, footprints:Pin_Header_Straight_2x03, symbol formula:CONN_02X03
Changed lines of the file:
@@
 	1    0    0    -1
 $EndComp
-Text Label 1375 2650 0    50   ~ 0
-MISO
-Text Label 1375 2750 0    50   ~ 0
-SCK
-Text Label 1375 2850 0    50   ~ 0
-RESET
-Text Label 1375 3050 0    50   ~ 0
-MOSI
 Wire Wire Line
 	9125 2925 9125 2825
@@
 NoConn ~ 2350 5775
 NoConn ~ 11050 6725
-$Comp
-L rocketry:USB_MicroB U5
-U 1 1 5C686BB4
-P 1075 2650
-F 0 "U5" H 1130 3117 50  0000 C CNN
-F 1 "USB_MicroB" H 1130 3026 50  0000 C CNN
-F 2 "Connectors_USB:USB_Micro-B_Molex-105017-0001" H 1025 3000 50  0001 C CNN
-F 3 "https://www.molex.com/pdm_docs/sd/1050170001_sd.pdf" H 1025 3000 50  0001 C CNN
-F 4 "DK" H 1325 2400 50  0001 C CNN "MFN"
-F 5 "WM1399CT-ND" H 1425 2500 50  0001 C CNN "MPN"
-F 6 "https://www.digikey.com/product-detail/en/molex-llc/1050170001/WM1399CT-ND/2350885" H 1525 2600 50  0001 C CNN "PurchasingLink"
-	1    1075 2650
-	1    0    0    -1
-$EndComp
-Wire Wire Line
-	1075 3050 1375 3050
-Wire Wire Line
-	975  3050 975  3125
-$Comp
-L power:GND #PWR01
-U 1 1 5C68DB3A
-P 975 3125
-F 0 "#PWR01" H 975 2875 50  0001 C CNN
-F 1 "GND" H 980 2952 50  0000 C CNN
-F 2 "" H 975 3125 50  0001 C CNN
-F 3 "" H 975 3125 50  0001 C CNN
-	1    975  3125
-	1    0    0    -1
-$EndComp
 Wire Wire Line
 	4075 2750 4075 2850
@@
 	1    0    0    -1
 $EndComp
-$Comp
-L power:VCC #PWR06
-U 1 1 5CB8C32E
-P 1625 2375
-F 0 "#PWR06" H 1625 2225 50  0001 C CNN
-F 1 "VCC" H 1642 2548 50  0000 C CNN
-F 2 "" H 1625 2375 50  0001 C CNN
-F 3 "" H 1625 2375 50  0001 C CNN
-	1    1625 2375
-	1    0    0    -1
-$EndComp
-Wire Wire Line
-	1625 2450 1625 2375
-Wire Wire Line
-	1375 2450 1625 2450
 Text Label 9825 1525 2    50   ~ 0
 Dectect_LED
@@
 Text Label 5525 2700 0    50   ~ 0
 SCL
+$Comp
+L power:VCC #PWR06
+U 1 1 5CB8C32E
+P 2200 2900
+F 0 "#PWR06" H 2200 2750 50  0001 C CNN
+F 1 "VCC" H 2217 3073 50  0000 C CNN
+F 2 "" H 2200 2900 50  0001 C CNN
+F 3 "" H 2200 2900 50  0001 C CNN
+	1    2200 2900
+	1    0    0    -1
+$EndComp
+$Comp
+L power:GND #PWR01
+U 1 1 5C68DB3A
+P 2150 3550
+F 0 "#PWR01" H 2150 3300 50  0001 C CNN
+F 1 "GND" H 2155 3377 50  0000 C CNN
+F 2 "" H 2150 3550 50  0001 C CNN
+F 3 "" H 2150 3550 50  0001 C CNN
+	1    2150 3550
+	1    0    0    -1
+$EndComp
+Text Label 2000 3350 0    50   ~ 0
+MOSI
+Text Label 1500 3450 2    50   ~ 0
+RESET
+Text Label 1500 3350 2    50   ~ 0
+SCK
+Text Label 1500 3250 2    50   ~ 0
+MISO
+$Comp
+L formula:CONN_02X03 J2
+U 1 1 5CE52224
+P 1750 3350
+F 0 "J2" H 1750 3665 50  0000 C CNN
+F 1 "CONN_02X03" H 1750 3574 50  0000 C CNN
+F 2 "footprints:Pin_Header_Straight_2x03" H 1750 2150 50  0001 C CNN
+F 3 "http://portal.fciconnect.com/Comergent//fci/drawing/67996.pdf" H 1750 2150 50  0001 C CNN
+F 4 "DK" H 1750 3350 60  0001 C CNN "MFN"
+F 5 "609-3234-ND" H 1750 3350 60  0001 C CNN "MPN"
+F 6 "https://www.digikey.com/product-detail/en/amphenol-fci/67997-206HLF/609-3234-ND/1878491" H 2150 3950 60  0001 C CNN "PurchasingLink"
+	1    1750 3350
+	1    0    0    -1
+$EndComp
+Wire Wire Line
+	2000 3250 2200 3250
+Wire Wire Line
+	2200 3250 2200 2900
+Wire Wire Line
+	2000 3450 2150 3450
+Wire Wire Line
+	2150 3450 2150 3550
 $EndSCHEMATC
