File: circuit/circuit.kicad_pcb (KiCad board)
At the start: 2 copper layers, 30 x 40 mm, 30 parts, among them J1 JST-PH_2_RA, U1 SK812, U2 LM1117MPX-3.3, U3 ADXL345, U4 ATmega328-AU, U5 USB_MicroB, Y1 Crystal_SMD

Commit message: pushing but not done
Parts:
- moved C8 9.23 mm to (186.7, 85.9)
- moved C9 3.49 mm to (189.5, 85.2)
- moved R9 2.60 mm to (192.3, 84.9)
- moved U2 1.82 mm to (206.1, 92.2)
Routing:
- net VCC: track 93.0 -> 47.1 mm, vias 6 -> 4
- net GND: track 69.0 -> 97.9 mm, vias 15 -> 16
- net /MISO: track 0.00 -> 22.6 mm, vias 0 -> 1
- net /SCK: track 0.00 -> 22.3 mm, vias 0 -> 1
- net /MOSI: track 0.00 -> 20.8 mm, vias 0 -> 1
- net Net-(R9-Pad2): track 4.19 -> 0.00 mm
